File: motor_controller.kicad_pcb (KiCad board)
At the start: 2 copper layers, 76.2 x 50.8 mm, 32 parts, among them J1 Conn_01x03_Pin, J2 POWER, J5 To RPico, Q1 IPP040N06NF2S, Q2 IPP040N06NF2S, Q3 IPP040N06NF2S, Q4 IPP040N06NF2S, Q5 IPP040N06NF2S, Q6 IPP040N06NF2S, U1 A5932

Commit message: Add files via upload
Parts:
- moved J2 63.1 mm to (212.5, 31.1)
- moved R1 62.0 mm to (273.7, 58.0)
- moved R10 46.4 mm to (267.5, 45.0)
- moved Q1 35.1 mm to (272.7, 40.0), turned to 180 degrees
- moved R11 32.8 mm to (249.6, 41.9), turned to 90 degrees
- moved Q4 27.6 mm to (267.6, 55.0), turned to 0 degrees
- moved R8 27.2 mm to (216.5, 43.7), turned to 90 degrees
- moved J1 25.6 mm to (251.4, 70.0), turned to 0 degrees
- moved J5 25.4 mm to (207.0, 55.4), turned to 180 degrees
- moved R12 24.5 mm to (234.8, 42.7), turned to 90 degrees
- moved R15 22.6 mm to (236.0, 54.5), turned to -90 degrees
- moved R9 22.3 mm to (221.0, 53.0), turned to 90 degrees
- moved C6 21.6 mm to (220.8, 43.7), turned to -90 degrees
- moved R6 21.0 mm to (212.3, 43.7), turned to -90 degrees
- moved C4 20.4 mm to (230.3, 43.5)
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Connections:
- Q1 pad 3: Net-(J1-Pin_1) -> Net-(J1-Pin_3)
- Q3 pad 3: Net-(J1-Pin_3) -> Net-(J1-Pin_1)
- Q4 pad 2: Net-(J1-Pin_1) -> Net-(J1-Pin_3)
- Q6 pad 2: Net-(J1-Pin_3) -> Net-(J1-Pin_1)
- U1 pad 16: Net-(J1-Pin_1) -> Net-(J1-Pin_3)
- U1 pad 20: Net-(J1-Pin_3) -> Net-(J1-Pin_1)
Routing:
- net Net-(J1-Pin_3): track 1.31 -> 72.1 mm, vias 0 -> 1
- net Net-(J1-Pin_2): track 0.00 -> 56.1 mm, vias 0 -> 1
- net Net-(Q4-S): track 0.00 -> 56.1 mm
- net GND: track 0.00 -> 52.2 mm, vias 0 -> 5
- net Net-(J1-Pin_1): track 0.00 -> 44.3 mm, vias 0 -> 1
- net Net-(U1-GHA): track 0.00 -> 37.2 mm
- net Net-(Q4-G): track 0.00 -> 34.9 mm
- net Net-(U1-SPD): track 0.00 -> 27.2 mm, vias 0 -> 1
- net DIR: track 0.00 -> 26.4 mm, vias 0 -> 2
- net VIN: track 0.00 -> 24.5 mm
- net Net-(U1-GHB): track 0.00 -> 22.3 mm
- net BRAKE: track 0.00 -> 21.1 mm, vias 0 -> 2
- net Net-(Q5-G): track 0.00 -> 20.4 mm
- net Net-(U1-FG): track 0.00 -> 16.5 mm
- net Net-(U1-VREF): track 0.00 -> 16.0 mm
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- added copper zone on B.Cu, net GND
- added copper zone on F.Cu, net VIN

Commit message: Add files via upload
Parts:
- removed R1: R_Small, Resistor_SMD:R_0805_2012Metric_Pad1.20x1.40mm_HandSolder
- C1, C2: value C_Small -> 100u; footprint Capacitor_SMD:C_0805_2012Metric_Pad1.18x1.45mm_HandSolder -> Capacitor_THT:C_Radial_D5.0mm_H7.0mm_P2.00mm
- D1: footprint LED_SMD:LED_0805_2012Metric_Pad1.15x1.40mm_HandSolder -> LED_THT:LED_D5.0mm
- R10, R11, R12, R13, R14, R15: value R_Small -> 2.2; footprint Resistor_SMD:R_0805_2012Metric_Pad1.20x1.40mm_HandSolder -> Resistor_THT:R_Axial_DIN0207_L6.3mm_D2.5mm_P7.62mm_Horizontal
- R2: value R_Small -> 30k; footprint Resistor_SMD:R_0805_2012Metric_Pad1.20x1.40mm_HandSolder -> Resistor_THT:R_Axial_DIN0207_L6.3mm_D2.5mm_P7.62mm_Horizontal
- R3, R5, R7: value R_Small -> 10k; footprint Resistor_SMD:R_0805_2012Metric_Pad1.20x1.40mm_HandSolder -> Resistor_THT:R_Axial_DIN0207_L6.3mm_D2.5mm_P7.62mm_Horizontal
- R4: value R_Small -> 220; footprint Resistor_SMD:R_0805_2012Metric_Pad1.20x1.40mm_HandSolder -> Resistor_THT:R_Axial_DIN0207_L6.3mm_D2.5mm_P7.62mm_Horizontal
- R6: footprint Resistor_SMD:R_0805_2012Metric_Pad1.20x1.40mm_HandSolder -> Resistor_THT:R_Axial_DIN0207_L6.3mm_D2.5mm_P7.62mm_Horizontal
- R8: value R_Small -> 10k; footprint Resistor_SMD:R_0805_2012Metric_Pad1.20x1.40mm_HandSolder -> Resistor_THT:R_Axial_DIN0207_L6.3mm_D2.5mm_P7.62mm_Horizontal; moved to B.Cu
- R9: value R_Small -> 330; footprint Resistor_SMD:R_0805_2012Metric_Pad1.20x1.40mm_HandSolder -> Resistor_THT:R_Axial_DIN0207_L6.3mm_D2.5mm_P7.62mm_Horizontal
- moved C1 143.6 mm to (90.0, 69.8), turned to 180 degrees
- moved C2 142.4 mm to (90.0, 76.2), turned to 180 degrees
- moved J2 126.6 mm to (88.6, 57.0)
- moved R8 122.8 mm to (103.5, 91.8)
- moved R3 118.6 mm to (103.5, 72.2), turned to 0 degrees
- moved R5 115.5 mm to (103.4, 75.8), turned to 0 degrees
- moved R6 114.5 mm to (103.4, 79.2), turned to 0 degrees
- moved J5 112.4 mm to (103.4, 99.2), turned to 90 degrees
- moved R10 110.4 mm to (160.9, 73.8)
- moved R7 110.0 mm to (111.0, 95.2), turned to 0 degrees
- moved R9 109.2 mm to (118.0, 89.3)
- moved R11 108.4 mm to (144.7, 69.5), turned to 0 degrees
- moved R2 105.9 mm to (121.4, 81.7)
- moved C6 105.8 mm to (118.5, 71.0)
- moved C4 105.2 mm to (128.7, 71.0)
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Connections:
- Q4 pad 3: Net-(Q4-S) -> GND
- Q5 pad 3: Net-(Q4-S) -> GND
- Q6 pad 3: Net-(Q4-S) -> GND
- U1 pad 15: Net-(Q4-S) -> GND
Routing:
- net GND: track 52.2 -> 117.5 mm
- net Net-(Q4-S): track 56.1 -> 0.00 mm
- net Net-(J1-Pin_3): track 72.1 -> 113.4 mm
- net Net-(J1-Pin_2): track 56.1 -> 91.4 mm
- net PWM_in: track 3.21 -> 32.7 mm
- net Net-(J1-Pin_1): track 44.3 -> 67.1 mm
- net Net-(Q1-G): track 7.87 -> 30.4 mm, vias 0 -> 1
- net DIR: track 26.4 -> 47.4 mm, vias 2 -> 1
- net VIN: track 24.5 -> 45.0 mm
- net Net-(Q2-G): track 13.7 -> 30.1 mm
- net BRAKE: track 21.1 -> 36.5 mm, vias 2 -> 1
- net Net-(Q4-G): track 34.9 -> 46.8 mm
- net VREF: track 0.00 -> 11.9 mm
- net Net-(Q5-G): track 20.4 -> 30.3 mm
- net Net-(D1-A): track 2.91 -> 12.8 mm
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- added copper zone on F.Cu, net GND
Other:
- board size 76.2 x 50.8 mm -> 152.4 x 50.8 mm

Commit message: Add files via upload
Parts:
- removed J5: To RPico, Connector_PinSocket_2.54mm:PinSocket_1x04_P2.54mm_Vertical
- removed R5, R7: 10k, Resistor_THT:R_Axial_DIN0207_L6.3mm_D2.5mm_P7.62mm_Horizontal
- added J3: Conn_01x04_Pin, Connector_PinSocket_2.54mm:PinSocket_1x04_P2.54mm_Vertical, F.Cu at (101.0, 99.2)
- R8: moved to F.Cu
- moved R8 19.0 mm to (113.8, 75.9), turned to -90 degrees
- moved R4 14.9 mm to (101.0, 83.5), turned to 90 degrees
- moved R3 5.51 mm to (109.0, 72.7)
- moved R6 4.82 mm to (106.9, 75.9), turned to -90 degrees
- moved C6 2.06 mm to (119.0, 69.0)
Connections:
- net Net-(U1-FG) renamed FG
- R3 pad 1: VREF -> Net-(U1-VREF)
- R6 pad 1: VREF -> Net-(U1-VREF)
- R8 pad 2: VREF -> GND
- U1 pad 3: BRAKE -> GND
- U1 pad 7: Net-(U1-RD) -> unconnected-(U1-RD-Pad7)
Routing:
- net DIR: track 47.4 -> 10.2 mm, vias 1 -> 0
- net BRAKE: track 36.5 -> 0.00 mm, vias 1 -> 0
- net Net-(U1-VREF): track 7.30 -> 25.1 mm
- net PWM_in: track 32.7 -> 15.8 mm
- net Net-(U1-RD): track 13.3 -> 0.00 mm
- net Net-(U1-SPD): track 17.9 -> 30.9 mm
- net VREF: track 11.9 -> 0.00 mm
- net GND: track 117.5 -> 128.8 mm
- net Net-(J1-Pin_1): track 67.1 -> 70.3 mm
- net FG: track 13.8 -> 16.1 mm
- net Net-(J1-Pin_2): track 91.4 -> 90.6 mm
- net Net-(U1-GLC): track 9.66 -> 9.00 mm
- net Net-(U1-GHC): track 12.4 -> 13.1 mm
