File: motor_controller.kicad_sch (KiCad schematic)
At the start: 21 parts, among them J1 Conn_01x03_Pin, Q1 IPP040N06NF2S, Q2 IPP040N06NF2S, Q3 IPP040N06NF2S, Q4 IPP040N06NF2S, Q5 IPP040N06NF2S, Q6 IPP040N06NF2S, U2 RP2040

Commit message: Add files via upload
updated stuff
Parts:
- removed U2: RP2040, Package_DFN_QFN:QFN-56-1EP_7x7mm_P0.4mm_EP3.2x3.2mm, symbol MCU_RaspberryPi:RP2040
- added A1: RaspberryPi_Pico, Module:RaspberryPi_Pico_Common_Unspecified, symbol MCU_Module:RaspberryPi_Pico
- added J2: POWER, symbol Connector:Conn_01x02_Pin
- added J3: J_BUCK_IN, symbol Connector:Conn_01x02_Pin
- added J4: J_BUCK_OUT, symbol Connector:Conn_01x02_Pin
Connections:
- net GND: now also A1.13 (GND), A1.18 (GND), A1.23 (GND), A1.28 (GND), A1.3 (GND), A1.38 (GND), A1.8 (GND), J2.2 (Pin_2), J3.2 (Pin_2), J4.2 (Pin_2)
- net PWM_in: now also A1.1 (GPIO0)
- net VIN: now also J2.1 (Pin_1), J3.1 (Pin_1)
- net BRAKE: no longer names the net of U1.3 (BRAKE)
- net DIR: no longer names the net of U1.6 (DIR)
- net nFAULT: no longer names the net of U1.9 (nFAULT)
- new net 5V: A1.39 (VSYS), J4.1 (Pin_1)
- no-connect marks 1 -> 32
Other:
- note added: "LM2596S Buck Converter"
- note added: "PWM Input from RPI Pico"
- note added: "Power Stage"

Commit message: Add files via upload
Parts:
- removed A1: RaspberryPi_Pico, Module:RaspberryPi_Pico_Common_Unspecified, symbol MCU_Module:RaspberryPi_Pico
- removed J3: J_BUCK_IN, symbol Connector:Conn_01x02_Pin
- removed J4: J_BUCK_OUT, symbol Connector:Conn_01x02_Pin
- added D1: LED, LED_SMD:LED_0805_2012Metric_Pad1.15x1.40mm_HandSolder, symbol Device:LED
- added J5: To RPico, Connector_PinSocket_2.54mm:PinSocket_1x04_P2.54mm_Vertical, symbol Connector:Conn_01x04_Pin
- added R10, R11, R12, R13, R14, R15, R7, R8, R9: R_Small, Resistor_SMD:R_0805_2012Metric_Pad1.20x1.40mm_HandSolder, symbol Device:R_Small
- C1, C2, C3, C4, C5, C6: footprint (none) -> Capacitor_SMD:C_0805_2012Metric_Pad1.18x1.45mm_HandSolder
- J1: footprint (none) -> TerminalBlock_Phoenix:TerminalBlock_Phoenix_MKDS-1,5-3-5.08_1x03_P5.08mm_Horizontal
- J2: footprint (none) -> TerminalBlock_Phoenix:TerminalBlock_Phoenix_MKDS-1,5-2-5.08_1x02_P5.08mm_Horizontal
- Q1, Q2, Q3, Q4, Q5, Q6: footprint (none) -> Package_TO_SOT_THT:TO-220-3_Vertical
- R1, R2, R3, R4, R5: footprint (none) -> Resistor_SMD:R_0805_2012Metric_Pad1.20x1.40mm_HandSolder
- R6: value R_Small -> 10k; footprint (none) -> Resistor_SMD:R_0805_2012Metric_Pad1.20x1.40mm_HandSolder
- U1: value ~ -> A5932; footprint (none) -> Custom:HTSSOP-24-1EP_4.4x7.8mm_P0.65mm_EP3.4x4.75mm_Mask2.4x2.98mm
Connections:
- net GND: now also U1.25 (EP), D1.1 (K), J5.4 (Pin_4), R7.2
- net PWM_in: now also J5.1 (Pin_1)
- net VREF: now also R8.2
- net at Q5.1 (G): now also R14.2; no longer U1.13 (GLB)
- net at Q4.1 (G): now also R13.2; no longer U1.12 (GLA)
- net at Q1.1 (G): now also R10.2; no longer U1.17 (GHA)
- net at Q6.1 (G): now also R15.2; no longer U1.14 (GLC)
- net at U1.19 (GHB): now also R11.1; no longer Q2.1 (G)
- net at U1.21 (GHC): now also R12.1; no longer Q3.1 (G)
- net BRAKE: now reaches U1.3 (BRAKE)
- net BRAKE: now also J5.3 (Pin_3), R7.1
- net DIR: now reaches U1.6 (DIR)
- net DIR: now also J5.2 (Pin_2), R8.1
- net at U1.9 (nFAULT): now also R9.2
- new net: Q3.1 (G), R12.2
- new net: D1.2 (A), R9.1
- new net: R10.1, U1.17 (GHA)
- new net: Q2.1 (G), R11.2
- new net: R14.1, U1.13 (GLB)
- new net: R13.1, U1.12 (GLA)
- new net: R15.1, U1.14 (GLC)
- no-connect marks 32 -> 1
Other:
- note removed: "LM2596S Buck Converter"
- note removed: "PWM Input from RPI Pico"
- moved on the sheet: C1, C2, C3, C4, C5, C6, J1, J2, Q1, Q2, Q3, Q4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

Commit message: Add files via upload
holy larp
Parts:
- R10-2.2: renamed from R10; value R_Small -> 2.2
- R11-2.2: renamed from R11; value R_Small -> 2.2
- R12-2.2: renamed from R12; value R_Small -> 2.2
- R13-2.2: renamed from R13; value R_Small -> 2.2
- R14-2.2: renamed from R14; value R_Small -> 2.2
- R15-2.2: renamed from R15; value R_Small -> 2.2
- R2-15k: renamed from R2; value R_Small -> 15k
- R5-10k: renamed from R5; value R_Small -> 10k
- R7-10k: renamed from R7; value R_Small -> 10k
- R8-10k: renamed from R8; value R_Small -> 10k
- R9-330: renamed from R9; value R_Small -> 330
Other:
- moved on the sheet: C6

Commit message: Add files via upload
Parts:
- R10: renamed from R10-2.2; value 2.2 -> R_Small
- R11: renamed from R11-2.2; value 2.2 -> R_Small
- R12: renamed from R12-2.2; value 2.2 -> R_Small
- R13: renamed from R13-2.2; value 2.2 -> R_Small
- R14: renamed from R14-2.2; value 2.2 -> R_Small
- R15: renamed from R15-2.2; value 2.2 -> R_Small
- R2: renamed from R2-15k; value 15k -> R_Small
- R5: renamed from R5-10k; value 10k -> R_Small
- R7: renamed from R7-10k; value 10k -> R_Small
- R8: renamed from R8-10k; value 10k -> R_Small
- R9: renamed from R9-330; value 330 -> R_Small
Connections:
- net at Q1.3 (S), Q4.2 (D), U1.16 (SA): now also J1.3 (Pin_3); no longer J1.1 (Pin_1)
- net at Q3.3 (S), Q6.2 (D), U1.20 (SC): now also J1.1 (Pin_1); no longer J1.3 (Pin_3)
Other:
- moved on the sheet: C6, J1
Changed lines of the file:
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@@
 	(wire
 		(pts
-			(xy 97.79 115.57) (xy 100.33 115.57)
+			(xy 100.33 115.57) (xy 97.79 115.57)
 		)
 		(stroke
@@
 	(wire
 		(pts
-			(xy 95.25 129.54) (xy 99.06 129.54)
+			(xy 95.25 129.54) (xy 100.33 129.54)
 		)
 		(stroke
@@
 	(wire
 		(pts
-			(xy 104.14 129.54) (xy 109.22 129.54)
+			(xy 105.41 129.54) (xy 109.22 129.54)
 		)
 		(stroke
@@
 		(in_pos_files yes)
 		(dnp no)
-		(property "Reference" "R12-2.2"
+		(property "Reference" "R12"
 			(at 169.164 81.026 0)
 			(show_name no)
@@
 			)
 		)
-		(property "Value" "2.2"
+		(property "Value" "R_Small"
 			(at 167.6399 74.93 0)
 			(hide yes)
@@
 			(project "motor_controller"
 				(path "/be9826e1-4220-47d5-9f24-2299ce8144d5"
-					(reference "R12-2.2")
+					(reference "R12")
 					(unit 1)
 				)
@@
 		(in_pos_files yes)
 		(dnp no)
-		(property "Reference" "R10-2.2"
+		(property "Reference" "R10"
 			(at 169.164 73.152 0)
 			(show_name no)
@@
 			)
 		)
-		(property "Value" "2.2"
+		(property "Value" "R_Small"
 			(at 167.6399 67.31 0)
 			(hide yes)
@@
 			(project "motor_controller"
 				(path "/be9826e1-4220-47d5-9f24-2299ce8144d5"
-					(reference "R10-2.2")
+					(reference "R10")
 					(unit 1)
 				)
@@
 		(in_pos_files yes)
 		(dnp no)
-		(property "Reference" "R11-2.2"
+		(property "Reference" "R11"
 			(at 169.164 76.962 0)
 			(show_name no)
@@
 			)
 		)
-		(property "Value" "2.2"
+		(property "Value" "R_Small"
 			(at 167.6399 71.12 0)
 			(hide yes)
@@
 			(project "motor_controller"
 				(path "/be9826e1-4220-47d5-9f24-2299ce8144d5"
-					(reference "R11-2.2")
+					(reference "R11")
 					(unit 1)
 				)
@@
 		(in_pos_files yes)
 		(dnp no)
-		(property "Reference" "R14-2.2"
+		(property "Reference" "R14"
 			(at 169.418 103.886 0)
 			(show_name no)
@@
 			)
 		)
-		(property "Value" "2.2"
+		(property "Value" "R_Small"
 			(at 167.6399 97.79 0)
 			(hide yes)
@@
 			(project "motor_controller"
 				(path "/be9826e1-4220-47d5-9f24-2299ce8144d5"
-					(reference "R14-2.2")
+					(reference "R14")
 					(unit 1)
 				)
@@
 		(in_pos_files yes)
 		(dnp no)
-		(property "Reference" "R5-10k"
+		(property "Reference" "R5"
 			(at 93.218 93.726 0)
 			(show_name no)
@@
 			)
 		)
-		(property "Value" "10k"
+		(property "Value" "R_Small"
 			(at 93.98 95.2499 0)
 			(hide yes)
@@
 			(project "motor_controller"
 				(path "/be9826e1-4220-47d5-9f24-2299ce8144d5"
-					(reference "R5-10k")
+					(reference "R5")
 					(unit 1)
 				)
@@
 	(symbol
 		(lib_id "Connector:Conn_01x03_Pin")
-		(at 234.95 87.63 0)
-		(mirror y)
+		(at 234.95 87.63 180)
 		(unit 1)
 		(body_style 1)
@@
 		(dnp no)
 		(property "Reference" "J1"
-			(at 234.315 80.01 0)
+			(at 234.315 95.25 0)
 			(show_name no)
 			(do_not_autoplace no)
@@
 		)
 		(property "Value" "Conn_01x03_Pin"
-			(at 234.315 82.55 0)
+			(at 234.315 92.71 0)
 			(show_name no)
 			(do_not_autoplace no)
@@
 		(in_pos_files yes)
 		(dnp no)
-		(property "Reference" "R13-2.2"
+		(property "Reference" "R13"
 			(at 169.418 99.822 0)
 			(show_name no)
@@
 			)
 		)
-		(property "Value" "2.2"
+		(property "Value" "R_Small"
 			(at 167.6399 93.98 0)
 			(hide yes)
@@
 			(project "motor_controller"
 				(path "/be9826e1-4220-47d5-9f24-2299ce8144d5"
-					(reference "R13-2.2")
+					(reference "R13")
 					(unit 1)
 				)
@@
 		(in_pos_files yes)
 		(dnp no)
-		(property "Reference" "R8-10k"
+		(property "Reference" "R8"
 			(at 72.898 86.106 0)
 			(show_name no)
@@
 			)
 		)
-		(property "Value" "10k"
+		(property "Value" "R_Small"
 			(at 73.66 87.6299 0)
 			(hide yes)
@@
 			(project "motor_controller"
 				(path "/be9826e1-4220-47d5-9f24-2299ce8144d5"
-					(reference "R8-10k")
+					(reference "R8")
 					(unit 1)
 				)
@@
 	(symbol
 		(lib_id "Device:C_Small")
-		(at 101.6 129.54 90)
+		(at 102.87 129.54 90)
 		(unit 1)
 		(body_style 1)
@@
 		(fields_autoplaced yes)
 		(property "Reference" "C6"
-			(at 101.6063 123.19 90)
+			(at 102.8763 123.19 90)
 			(show_name no)
 			(do_not_autoplace no)
@@
 		)
 		(property "Value" "0.1 uF X5R 10V"
-			(at 101.6063 125.73 90)
+			(at 102.8763 125.73 90)
 			(show_name no)
 			(do_not_autoplace no)
@@
 		)
 		(property "Footprint" "Capacitor_SMD:C_0805_2012Metric_Pad1.18x1.45mm_HandSolder"
-			(at 101.6 129.54 0)
+			(at 102.87 129.54 0)
 			(hide yes)
 			(show_name no)
@@
 		)
 		(property "Datasheet" ""
-			(at 101.6 129.54 0)
+			(at 102.87 129.54 0)
 			(hide yes)
 			(show_name no)
@@
 		)
 		(property "Description" "Unpolarized capacitor, small symbol"
-			(at 101.6 129.54 0)
+			(at 102.87 129.54 0)
 			(hide yes)
 			(show_name no)
@@
 		(in_pos_files yes)
 		(dnp no)
-		(property "Reference" "R9-330"
+		(property "Reference" "R9"
 			(at 102.616 113.792 0)
 			(show_name no)
@@
 			)
 		)
-		(property "Value" "330"
+		(property "Value" "R_Small"
 			(at 104.1399 113.03 0)
 			(hide yes)
@@
 			(project "motor_controller"
 				(path "/be9826e1-4220-47d5-9f24-2299ce8144d5"
-					(reference "R9-330")
+					(reference "R9")
 					(unit 1)
 				)
@@
 		(in_pos_files yes)
 		(dnp no)
-		(property "Reference" "R7-10k"
+		(property "Reference" "R7"
 			(at 66.548 88.646 0)
 			(show_name no)
@@
 			)
 		)
-		(property "Value" "10k"
+		(property "Value" "R_Small"
 			(at 67.31 90.1699 0)
 			(hide yes)
@@
 			(project "motor_controller"
 				(path "/be9826e1-4220-47d5-9f24-2299ce8144d5"
-					(reference "R7-10k")
+					(reference "R7")
 					(unit 1)
 				)
@@
 		(in_pos_files yes)
 		(dnp no)
-		(property "Reference" "R2-15k"
+		(property "Reference" "R2"
 			(at 161.036 121.412 0)
 			(show_name no)
@@
 			)
 		)
-		(property "Value" "15k"
+		(property "Value" "R_Small"
 			(at 162.5599 120.65 0)
 			(hide yes)
@@
 			(project "motor_controller"
 				(path "/be9826e1-4220-47d5-9f24-2299ce8144d5"
-					(reference "R2-15k")
+					(reference "R2")
 					(unit 1)
 				)
@@
 		(in_pos_files yes)
 		(dnp no)
-		(property "Reference" "R15-2.2"
+		(property "Reference" "R15"
 			(at 169.418 107.442 0)
 			(show_name no)
@@
 			)
 		)
-		(property "Value" "2.2"
+		(property "Value" "R_Small"
 			(at 167.6399 101.6 0)
 			(hide yes)
@@
 			(project "motor_controller"
 				(path "/be9826e1-4220-47d5-9f24-2299ce8144d5"
-					(reference "R15-2.2")
+					(reference "R15")
 					(unit 1)
 				)

Commit message: Add files via upload
Parts:
- removed R1: R_Small, Resistor_SMD:R_0805_2012Metric_Pad1.20x1.40mm_HandSolder, symbol Device:R_Small
- C1, C2: value C_Small -> 100u; footprint Capacitor_SMD:C_0805_2012Metric_Pad1.18x1.45mm_HandSolder -> Capacitor_THT:C_Radial_D5.0mm_H7.0mm_P2.00mm
- D1: footprint LED_SMD:LED_0805_2012Metric_Pad1.15x1.40mm_HandSolder -> LED_THT:LED_D5.0mm
- R10, R11, R12, R13, R14, R15: value R_Small -> 2.2; footprint Resistor_SMD:R_0805_2012Metric_Pad1.20x1.40mm_HandSolder -> Resistor_THT:R_Axial_DIN0207_L6.3mm_D2.5mm_P7.62mm_Horizontal
- R2: value R_Small -> 30k; footprint Resistor_SMD:R_0805_2012Metric_Pad1.20x1.40mm_HandSolder -> Resistor_THT:R_Axial_DIN0207_L6.3mm_D2.5mm_P7.62mm_Horizontal
- R3, R5, R7, R8: value R_Small -> 10k; footprint Resistor_SMD:R_0805_2012Metric_Pad1.20x1.40mm_HandSolder -> Resistor_THT:R_Axial_DIN0207_L6.3mm_D2.5mm_P7.62mm_Horizontal
- R4: value R_Small -> 220; footprint Resistor_SMD:R_0805_2012Metric_Pad1.20x1.40mm_HandSolder -> Resistor_THT:R_Axial_DIN0207_L6.3mm_D2.5mm_P7.62mm_Horizontal
- R6: footprint Resistor_SMD:R_0805_2012Metric_Pad1.20x1.40mm_HandSolder -> Resistor_THT:R_Axial_DIN0207_L6.3mm_D2.5mm_P7.62mm_Horizontal
- R9: value R_Small -> 330; footprint Resistor_SMD:R_0805_2012Metric_Pad1.20x1.40mm_HandSolder -> Resistor_THT:R_Axial_DIN0207_L6.3mm_D2.5mm_P7.62mm_Horizontal
Connections:
- net GND: now also Q4.3 (S), Q5.3 (S), Q6.3 (S), U1.15 (LSS)

Commit message: Add files via upload
Parts:
- removed J5: To RPico, Connector_PinSocket_2.54mm:PinSocket_1x04_P2.54mm_Vertical, symbol Connector:Conn_01x04_Pin
- removed R5, R7: 10k, Resistor_THT:R_Axial_DIN0207_L6.3mm_D2.5mm_P7.62mm_Horizontal, symbol Device:R_Small
- added J3: Conn_01x04_Pin, Connector_PinSocket_2.54mm:PinSocket_1x04_P2.54mm_Vertical, symbol Connector:Conn_01x04_Pin
Connections:
- net BRAKE is gone; now on net GND: U1.3 (BRAKE)
- net DIR: now also J3.2 (Pin_2)
- net GND: now also R8.2, J3.4 (Pin_4)
- net PWM_in: now also J3.1 (Pin_1)
- net VREF: no longer R8.2
- net FG: now reaches R6.2, U1.8 (FG)
- net FG: now also J3.3 (Pin_3)
- no-connect marks 1 -> 2
